File: Slim_Amp.kicad_pcb (KiCad board)
At the start: 4 copper layers, 65 x 82.5 mm, 52 parts, among them J1 Conn_Coaxial, J2 Bias_ctrl, J3 Conn_Coaxial, J4 Conn_01x04, Q1 ZVP2106G, Q2 RD07MUS2B, Q3 RD07MUS2B, T1 TLT, T2 BN61-202, U1 UA78M06CKVURG3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

Commit message: second commit
Parts:
- removed G***: LOGO, Athena:athena
- added J5: jumper, Connector_Molex:Molex_KK-254_AE-6410-02A_1x02_P2.54mm_Vertical, F.Cu at (93.4, 72.0)
- moved J2 3.21 mm to (93.3, 85.5)
- moved U2 1.74 mm to (108.9, 71.4)
Routing:
- net Net-(J2-Pin_1): track 21.7 -> 114.9 mm
- net Net-(Q2-D): track 0.00 -> 10.7 mm
- net Net-(J3-In): track 0.00 -> 10.5 mm
- net Net-(Q3-D): track 0.00 -> 10.5 mm
- net Net-(J5-Pin_2): track 12.1 -> 19.1 mm
- net Net-(Q3-G): track 4.47 -> 9.96 mm
- net Net-(Q2-G): track 4.44 -> 9.63 mm
- net Net-(T2-AA): track 0.00 -> 2.77 mm
- net Net-(T2-AB): track 0.00 -> 2.71 mm
- net Net-(C9-Pad1): track 0.00 -> 2.05 mm
- net GND: vias 0 -> 245
- removed copper zone on F.Cu, net Net-(J1-In)

Commit message: third commit
Parts:
- removed H1, H2: 3.3mm, MountingHole:MountingHole_3.2mm_M3_Pad_Via
- moved U2 2.00 mm to (106.9, 71.4)
Routing:
- net Net-(J5-Pin_2): track 19.1 -> 17.1 mm
- net Net-(J2-Pin_1): track 114.9 -> 113.2 mm
- net GND: vias 245 -> 246
Other:
- board size 65 x 82.5 mm -> 65 x 64.5 mm
- board text removed: "Il y a longtemps bien longtemps il y avait une bergère Qui gardait ses moutons bêlants dans une clairière Les moutons étaient tout crotés et la bergère était affreuse Laide les cheveux mal peignés et paresseuse Le fils du roi vint à passer C'était un parfait imbécile Il n'était ni beau ni bien fait Ni juvé ni juvé ni juvé-nile Et comme il était de surcroit myope comme une théière Il passa sans vo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"
- board text removed: "Laquelle à ce moment précis cherchait un pou dans son corsage Ce qui fait qu'elle ne le vit pas d'avantage Le fils du roi obtint la main d'une cousine abominable Et la bergère épousa un garçon dé garçon dé garçon d'étable Et tout s'étant ainsi passé suivant la plus saine logique Sans le concours d'aucune fée Aux dons magiques Il furent tous très malheureux et n'eurent pas un seul enfant C'est ain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"
