File: Slim_Amp.kicad_sch (KiCad schematic)
At the start: 51 parts, among them J1 Conn_Coaxial, J2 Bias_ctrl, J3 Conn_Coaxial, J4 Conn_01x04, Q1 ZVP2106G, Q2 RD07MUS2B, Q3 RD07MUS2B, T1 TLT, T2 BN61-202, U1 UA78M06CKVURG3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

Commit message: second commit
Parts:
- added J5: jumper, Connector_Molex:Molex_KK-254_AE-6410-02A_1x02_P2.54mm_Vertical, symbol Connector:Conn_01x02_Pin
Connections:
- net at C13.1, C14.1, C15.1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: now also J5.1 (Pin_1)
- net at C19.1, L1.2, U2.1 (VI): now also J5.2 (Pin_2)
Other:
- note added: "Jumper J5 si ddp trop faible"
Changed lines of the file:
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@@
 		)
 	)
+	(text "Jumper J5 si ddp trop faible"
+		(exclude_from_sim no)
+		(at 151.13 151.13 0)
+		(effects
+			(font
+				(size 1.27 1.27)
+			)
+		)
+	)
 	(junction
 		(at 97.79 161.29)
@@
 	(wire
 		(pts
+			(xy 165.1 124.46) (xy 165.1 132.08)
+		)
+		(stroke
+			(width 0)
+			(type default)
+		)
+	)
+	(wire
+		(pts
 			(xy 63.5 100.33) (xy 63.5 101.6)
 		)
@@
 	(wire
 		(pts
+			(xy 147.32 124.46) (xy 147.32 132.08)
+		)
+		(stroke
+			(width 0)
+			(type default)
+		)
+	)
+	(wire
+		(pts
 			(xy 137.16 99.06) (xy 137.16 100.33)
 		)
@@
 	(wire
 		(pts
+			(xy 156.21 124.46) (xy 165.1 124.46)
+		)
+		(stroke
+			(width 0)
+			(type default)
+		)
+	)
+	(wire
+		(pts
 			(xy 83.82 171.45) (xy 97.79 171.45)
 		)
@@
 	(wire
 		(pts
+			(xy 153.67 124.46) (xy 147.32 124.46)
+		)
+		(stroke
+			(width 0)
+			(type default)
+		)
+	)
+	(wire
+		(pts
 			(xy 105.41 69.85) (xy 105.41 72.39)
 		)
@@
 					(unit 1)
 				)
+			)
+		)
+	)
+	(symbol
+		(lib_id "Connector:Conn_01x02_Pin")
+		(at 153.67 119.38 90)
+		(mirror x)
+		(unit 1)
+		(body_style 1)
+		(exclude_from_sim no)
+		(in_bom yes)
+		(on_board yes)
+		(in_pos_files yes)
+		(dnp no)
+		(property "Reference" "J5"
+			(at 152.4 118.7449 90)
+			(show_name no)
+			(do_not_autoplace no)
+			(effects
+				(font
+					(size 1.27 1.27)
+				)
+				(justify left)
+			)
+		)
+		(property "Value" "jumper"
+			(at 152.4 121.2849 90)
+			(show_name no)
+			(do_not_autoplace no)
+			(effects
+				(font
+					(size 1.27 1.27)
+				)
+				(justify left)
+			)
+		)
+		(property "Footprint" "Connector_Molex:Molex_KK-254_AE-6410-02A_1x02_P2.54mm_Vertical"
+			(at 153.67 119.38 0)
+			(hide yes)
+			(show_name no)
+			(do_not_autoplace no)
+			(effects
+				(font
+					(size 1.27 1.27)
+				)
+			)
+		)
+		(property "Datasheet" ""
+			(at 153.67 119.38 0)
+			(hide yes)
+			(show_name no)
+			(do_not_autoplace no)
+			(effects
+				(font
+					(size 1.27 1.27)
+				)
+			)
+		)
+		(property "Description" "Generic connector, single row, 01x02, script generated"
+			(at 153.67 119.38 0)
+			(hide yes)
+			(show_name no)
+			(do_not_autoplace no)
+			(effects
+				(font
+					(size 1.27 1.27)
+				)
+			)
+		)
+		(pin "1"
+		)
+		(pin "2"
+		)
+		(instances
+			(project "Slim_Amp"
+				(path "/d2275eef-6863-4ebf-a9db-b7ee43970cb8"
+					(reference "J5")
+					(unit 1)
+				)

Commit message: third commit
Parts:
- removed H1, H2: 3.3mm, MountingHole:MountingHole_3.2mm_M3_Pad_Via, symbol Mechanical:MountingHole_Pad
